Commit message: updated

File: description/lidar.xacro (robot description, xacro)
@@ -4,4 +4,7 @@
         <visual>
             <geometry><mesh filename="package://jazzy_gz/meshes/lidar_link.STL" /></geometry>
+        <material name="light_black">
+        <color rgba="0.2 0.2 0.2 1.0" />
+        </material>
         </visual>
         <material name="red"/>
